File: HBL_2/VIBE/BASE/BASE.kicad_sch (KiCad schematic)
At the start: 27 parts, among them J1 QWIIC, J2 HUSB238, J3 HUSB238, J4 Ring_Conn, J5 Conn_01x02_Pin, J6 Conn_01x05_Socket, Q1 IRLZ14S, Q2 IRLZ14S, Q3 IRLZ14S, Q4 IRLZ14S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

Commit message: notes
Other:
- note added: "For haptic driver OR pressure sensor"
- note added: "Force sensitve resistor"
- note added: "Incremental Encoder"
- note added: "LED Ring molex con."
- note added: "Mosfets that ultimately goes to right side output"
- note added: "Usb-c power input module"
- note added: "Version 1, received May 12, 2025"
- note added: "force sensitive r."
Changed lines of the file:
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@@
 	(generator_version "9.0")
 	(paper "A4")
+	(text "Version 1, received May 12, 2025"
+		(exclude_from_sim no)
+		(at 197.866 170.18 0)
+		(effects
+			(font
+				(size 1.27 1.27)
+			)
+		)
+	)
+	(text "LED Ring molex con. "
+		(exclude_from_sim no)
+		(at 186.436 53.848 0)
+		(effects
+			(font
+				(size 1.27 1.27)
+			)
+		)
+	)
+	(text "For haptic driver OR pressure sensor"
+		(exclude_from_sim no)
+		(at 150.114 43.434 0)
+		(effects
+			(font
+				(size 1.27 1.27)
+			)
+		)
+	)
+	(text "force sensitive r."
+		(exclude_from_sim no)
+		(at 131.572 47.498 0)
+		(effects
+			(font
+				(size 1.27 1.27)
+			)
+		)
+	)
+	(text "Incremental Encoder"
+		(exclude_from_sim no)
+		(at 227.33 66.294 0)
+		(effects
+			(font
+				(size 1.27 1.27)
+			)
+		)
+	)
+	(text "Usb-c power input module"
+		(exclude_from_sim no)
+		(at 40.386 22.352 0)
+		(effects
+			(font
+				(size 1.27 1.27)
+			)
+		)
+	)
+	(text "Force sensitve resistor"
+		(exclude_from_sim no)
+		(at 266.954 46.482 0)
+		(effects
+			(font
+				(size 1.27 1.27)
+			)
+		)
+	)
+	(text "Mosfets that ultimately goes to right side output"
+		(exclude_from_sim no)
+		(at 232.41 90.424 0)
+		(effects
+			(font
+				(size 1.27 1.27)
+			)
+		)
+	)
 	(junction
 		(at 236.22 133.35)
